Commit message: got gazebo camera simulation working

File: urdf/controls/gazebo_sim_ros2_control.urdf.xacro (robot description, xacro)
@@ -7,4 +7,7 @@
                     <parameters>$(find vision_based_navigation_ttt)/config/control.yaml</parameters>
                 </plugin>
+                <plugin filename="gz-sim-sensors-system" name="gz::sim::systems::Sensors">
+                    <render_engine>ogre2</render_engine>
+                </plugin>
             </gazebo>
         </xacro:if>

File: urdf/jackal.urdf.xacro (robot description, xacro)
@@ -218,4 +218,66 @@
     <origin xyz="${mount_spacing} 0 0" />
   </joint>
+    <!-- STEP 7 - Camera -->
+    <joint type="fixed" name="camera_joint">
+      <origin xyz="0.225 0 0.075" rpy="0 0 0"/>
+      <child link="camera_link"/>
+      <parent link="base_link"/>
+      <axis xyz="0 1 0" />
+    </joint>
+    <link name='camera_link'>
+      <pose>0 0 0 0 0 0</pose>
+      <inertial>
+        <mass value="0.1"/>
+        <origin xyz="0 0 0" rpy="0 0 0"/>
+        <inertia
+            ixx="1e-6" ixy="0" ixz="0"
+            iyy="1e-6" iyz="0"
+            izz="1e-6"
+        />
+      </inertial>
+      <collision name='collision'>
+        <origin xyz="0 0 0" rpy="0 0 0"/>
+        <geometry>
+          <box size=".03 .03 .03"/>
+        </geometry>
+      </collision>
+      <visual name='camera_link_visual'>
+        <origin xyz="0 0 0" rpy="0 0 0"/>
+        <geometry>
+          <box size=".03 .03 .03"/>
+        </geometry>
+      </visual>
+    </link>
+    <gazebo reference="camera_link">
+      <material>Gazebo/Red</material>
+    </gazebo>
+    <gazebo reference="camera_link">
+      <sensor name="camera" type="camera">
+        <pose>0 0 0 0 0 0</pose>
+        <camera>
+          <horizontal_fov>1.3962634</horizontal_fov>
+          <image>
+            <width>640</width>
+            <height>480</height>
+            <format>R8G8B8</format>
+          </image>
+          <clip>
+            <near>0.1</near>
+            <far>15</far>
+          </clip>
+        </camera>
+        <always_on>true</always_on>
+        <update_rate>30</update_rate>
+        <visualize>true</visualize>
+        <topic>/camera/image</topic>
+      </sensor>
+    </gazebo>
+    <joint type="fixed" name="camera_optical_joint">
+      <origin xyz="0 0 0" rpy="-1.5707 0 -1.5707"/>
+      <child link="camera_link_optical"/>
+      <parent link="camera_link"/>
+    </joint>
+    <link name="camera_link_optical">
+    </link>
   <!-- Bring in simulation data for Gazebo. -->
   <!-- Optional standard accessories, including their simulation data. The rendering
