Commit message: got the jackal to move

File: urdf/controls/jackal_ros2_control.urdf.xacro (robot description, xacro)
@@ -8,65 +8,35 @@
       <!-- Define velocity control for all 4 wheels -->
       <joint name="front_left_wheel">
-        <command_interface name="velocity"/>
-        <state_interface name="position"/>
+        <command_interface name="velocity">
+          <param name="min">-10</param>
+          <param name="max">10</param>
+        </command_interface>               <state_interface name="position"/>
         <state_interface name="velocity"/>
       </joint>
       <joint name="front_right_wheel">
-        <command_interface name="velocity"/>
+        <command_interface name="velocity">
+          <param name="min">-10</param>
+          <param name="max">10</param>
+        </command_interface>
         <state_interface name="position"/>
         <state_interface name="velocity"/>
       </joint>
       <joint name="rear_left_wheel">
-        <command_interface name="velocity"/>
+        <command_interface name="velocity">
+          <param name="min">-10</param>
+          <param name="max">10</param>
+        </command_interface>
         <state_interface name="position"/>
         <state_interface name="velocity"/>
-      </joint>
+     </joint>
       <joint name="rear_right_wheel">
-        <command_interface name="velocity"/>
-        <state_interface name="position"/>
+        <command_interface name="velocity">
+          <param name="min">-10</param>
+          <param name="max">10</param>
+        </command_interface>               <state_interface name="position"/>
         <state_interface name="velocity"/>
       </joint>
     </ros2_control>
     <!-- 🔧 Add required transmissions for each wheel -->
-    <transmission name="trans_front_left_wheel">
-      <type>transmission_interface/SimpleTransmission</type>
-      <joint name="front_left_wheel">
-        <hardwareInterface>hardware_interface/VelocityJointInterface</hardwareInterface>
-      </joint>
-      <actuator name="front_left_motor">
-        <hardwareInterface>hardware_interface/VelocityJointInterface</hardwareInterface>
-        <mechanicalReduction>1</mechanicalReduction>
-      </actuator>
-    </transmission>
-    <transmission name="trans_front_right_wheel">
-      <type>transmission_interface/SimpleTransmission</type>
-      <joint name="front_right_wheel">
-        <hardwareInterface>hardware_interface/VelocityJointInterface</hardwareInterface>
-      </joint>
-      <actuator name="front_right_motor">
-        <hardwareInterface>hardware_interface/VelocityJointInterface</hardwareInterface>
-        <mechanicalReduction>1</mechanicalReduction>
-      </actuator>
-    </transmission>
-    <transmission name="trans_rear_left_wheel">
-      <type>transmission_interface/SimpleTransmission</type>
-      <joint name="rear_left_wheel">
-        <hardwareInterface>hardware_interface/VelocityJointInterface</hardwareInterface>
-      </joint>
-      <actuator name="rear_left_motor">
-        <hardwareInterface>hardware_interface/VelocityJointInterface</hardwareInterface>
-        <mechanicalReduction>1</mechanicalReduction>
-      </actuator>
-    </transmission>
-    <transmission name="trans_rear_right_wheel">
-      <type>transmission_interface/SimpleTransmission</type>
-      <joint name="rear_right_wheel">
-        <hardwareInterface>hardware_interface/VelocityJointInterface</hardwareInterface>
-      </joint>
-      <actuator name="rear_right_motor">
-        <hardwareInterface>hardware_interface/VelocityJointInterface</hardwareInterface>
-        <mechanicalReduction>1</mechanicalReduction>
-      </actuator>
-    </transmission>
   </xacro:macro>
 </robot>

Commit message: slight corridor_2 improvement

File: urdf/controls/jackal_ros2_control.urdf.xacro (robot description, xacro)
@@ -2,41 +2,85 @@
 <robot xmlns:xacro="http://www.ros.org/wiki/xacro">
   <xacro:macro name="jackal_ros2_control" params="use_gazebo">
-    <ros2_control name="GazeboSystem" type="system">
-      <hardware>
-        <plugin>gz_ros2_control/GazeboSimSystem</plugin>
-      </hardware>
-      <!-- Define velocity control for all 4 wheels -->
-      <joint name="front_left_wheel">
-        <command_interface name="velocity">
-          <param name="min">-10</param>
-          <param name="max">10</param>
-        </command_interface>               <state_interface name="position"/>
-        <state_interface name="velocity"/>
-      </joint>
-      <joint name="front_right_wheel">
-        <command_interface name="velocity">
-          <param name="min">-10</param>
-          <param name="max">10</param>
-        </command_interface>
-        <state_interface name="position"/>
-        <state_interface name="velocity"/>
-      </joint>
-      <joint name="rear_left_wheel">
-        <command_interface name="velocity">
-          <param name="min">-10</param>
-          <param name="max">10</param>
-        </command_interface>
-        <state_interface name="position"/>
-        <state_interface name="velocity"/>
-     </joint>
-      <joint name="rear_right_wheel">
-        <command_interface name="velocity">
-          <param name="min">-10</param>
-          <param name="max">10</param>
-        </command_interface>               <state_interface name="position"/>
-        <state_interface name="velocity"/>
-      </joint>
-    </ros2_control>
-    <!-- 🔧 Add required transmissions for each wheel -->
+    <xacro:if value="${use_gazebo}">
+      <ros2_control name="GazeboSystem" type="system">
+        <hardware>
+          <plugin>gz_ros2_control/GazeboSimSystem</plugin>
+        </hardware>
+        <!-- Define velocity control for all 4 wheels -->
+        <joint name="front_left_wheel">
+          <command_interface name="velocity">
+            <param name="min">-100</param>
+            <param name="max">100</param>
+          </command_interface>
+          <state_interface name="position"/>
+          <state_interface name="velocity"/>
+        </joint>
+        <joint name="front_right_wheel">
+          <command_interface name="velocity">
+            <param name="min">-100</param>
+            <param name="max">100</param>
+          </command_interface>
+          <state_interface name="position"/>
+          <state_interface name="velocity"/>
+        </joint>
+        <joint name="rear_left_wheel">
+          <command_interface name="velocity">
+            <param name="min">-100</param>
+            <param name="max">100</param>
+          </command_interface>
+          <state_interface name="position"/>
+          <state_interface name="velocity"/>
+        </joint>
+        <joint name="rear_right_wheel">
+          <command_interface name="velocity">
+            <param name="min">-100</param>
+            <param name="max">100</param>
+          </command_interface>
+          <state_interface name="position"/>
+          <state_interface name="velocity"/>
+        </joint>
+      </ros2_control>
+    </xacro:if>
+    <xacro:unless value="${use_gazebo}">
+      <ros2_control name="JackalSystem" type="system">
+        <hardware>
+          <plugin>jackal_base/JackalSystemHardware</plugin>
+        </hardware>
+        <param name="serial_port">/dev/ttyACM0</param>
+        <!-- Define velocity control for all 4 wheels -->
+        <joint name="front_left_wheel">
+          <command_interface name="velocity">
+            <param name="min">-10</param>
+            <param name="max">10</param>
+          </command_interface>
+          <state_interface name="position"/>
+          <state_interface name="velocity"/>
+        </joint>
+        <joint name="front_right_wheel">
+          <command_interface name="velocity">
+            <param name="min">-10</param>
+            <param name="max">10</param>
+          </command_interface>
+          <state_interface name="position"/>
+          <state_interface name="velocity"/>
+        </joint>
+        <joint name="rear_left_wheel">
+          <command_interface name="velocity">
+            <param name="min">-10</param>
+            <param name="max">10</param>
+          </command_interface>
+          <state_interface name="position"/>
+          <state_interface name="velocity"/>
+        </joint>
+        <joint name="rear_right_wheel">
+          <command_interface name="velocity">
+            <param name="min">-10</param>
+            <param name="max">10</param>
+          </command_interface>
+          <state_interface name="position"/>
+          <state_interface name="velocity"/>
+        </joint>
+      </ros2_control>
+    </xacro:unless>
   </xacro:macro>
 </robot>
