Commit message: Added meshes folder, updated README, CMAKE and jackal urdf file

File: urdf/jackal.urdf.xacro (robot description, xacro)
@@ -22,5 +22,5 @@
         <origin xyz="0 0 0" rpy="${PI/2} 0 0"/>
         <geometry>
-          <mesh filename="file://$(find jackal_description)/meshes/jackal-wheel.stl"/>
+          <mesh filename="file://$(find vision_based_navigation_ttt)/meshes/jackal-wheel.stl"/>
         </geometry>
         <material name="black" />
@@ -90,5 +90,5 @@
       <origin xyz="0 0 ${footprint_vertical_offset}" rpy="${PI/2} 0 ${PI/2}"/>
       <geometry>
-        <mesh filename="file://$(find jackal_description)/meshes/jackal-base.stl"/>
+        <mesh filename="file://$(find vision_based_navigation_ttt)/meshes/jackal-base.stl"/>
       </geometry>
       <material name="dark_grey" />
@@ -115,5 +115,5 @@
       <visual>
         <geometry>
-          <mesh filename="file://$(find jackal_description)/meshes/jackal-fender.stl"/>
+          <mesh filename="file://$(find vision_based_navigation_ttt)/meshes/jackal-fender.stl"/>
         </geometry>
         <material name="yellow" />
@@ -125,5 +125,5 @@
       <visual>
         <geometry>
-          <mesh filename="file://$(find jackal_description)/meshes/accessory_fender.stl"/>
+          <mesh filename="file://$(find vision_based_navigation_ttt)/meshes/accessory_fender.stl"/>
         </geometry>
         <material name="yellow" />
@@ -146,5 +146,5 @@
       <visual>
         <geometry>
-          <mesh filename="file://$(find jackal_description)/meshes/jackal-fender.stl"/>
+          <mesh filename="file://$(find vision_based_navigation_ttt)/meshes/jackal-fender.stl"/>
         </geometry>
         <material name="yellow" />
@@ -156,5 +156,5 @@
       <visual>
         <geometry>
-          <mesh filename="file://$(find jackal_description)/meshes/accessory_fender.stl"/>
+          <mesh filename="file://$(find vision_based_navigation_ttt)/meshes/accessory_fender.stl"/>
         </geometry>
         <material name="yellow" />
